File: HW/Kicad_files/wled_V1/wled_V1.kicad_pcb (KiCad board)
At the start: 2 copper layers, 32 parts, among them U3 TXS0102DCT

Commit message: routing update
Parts:
- 0440007.WRA1, C15, C5, C8: moved to B.Cu
- ESP32-S3-WROOM-1-N8: footprint Espressif:ESP32-S3-WROOM-1 -> SamacSys_Parts:ESP32S3WROOM1N8R8
- TSR-1-2450: footprint Package_TO_SOT_SMD:TO-252-3_TabPin2 -> SamacSys_Parts:TSR12450
- moved 39-30-3041 72.7 mm to (135.5, 82.8)
- moved 39-30-3041-bis1 71.7 mm to (135.5, 113.2)
- moved 0440007.WRA1 69.6 mm to (114.3, 127.0)
- moved C5 67.1 mm to (142.2, 120.2), turned to -90 degrees
- moved TP2 66.5 mm to (127.0, 105.7)
- moved TP3 66.5 mm to (127.0, 109.7)
- moved TP1 66.5 mm to (127.0, 101.6)
- moved TP6 66.5 mm to (131.1, 105.7)
- moved TP7 66.5 mm to (131.1, 109.7)
- moved TP5 66.5 mm to (131.1, 101.6)
- moved PJ-057AH1 63.7 mm to (111.8, 131.4), turned to 90 degrees
- moved U3 57.7 mm to (126.2, 117.8), turned to 180 degrees
- moved TP4 55.4 mm to (121.9, 101.6)
- moved JP1 46.4 mm to (132.1, 116.2), turned to 90 degrees
- moved 10164359-00011LF1 41.3 mm to (127.8, 141.4)
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