File: HW/wled_V1/wled_V1.kicad_sch (KiCad schematic)
At the start: 32 parts, among them U3 TXS0102DCT

Commit message: routing
Parts:
- removed 0440007.WRA1: Fuse, SamacSys_Parts:FUSC3216X85N, symbol Device:Fuse
- removed TP1, TP2, TP3, TP4, TP5, TP6, TP7: TestPoint, TestPoint:TestPoint_THTPad_2.0x2.0mm_Drill1.0mm, symbol Connector:TestPoint
- added J1: 0031.8201, SamacSys_Parts:0031.8201, symbol SamacSys_Parts:0031.8201
- 216990-0002: renamed from 10164359-00011LF1; footprint SamacSys_Parts:1016435900011LF -> SamacSys_Parts:2169900002; symbol Connector:USB_C_Receptacle -> SamacSys_Parts:216990-0002; Height (none) -> 3.36; Manufacturer_Name (none) -> Molex; Manufacturer_Part_Number (none) -> 216990-0002; Mouser Part Number (none) -> 538-216990-0002; Mouser Price/Stock (none) -> https://www.mouser.co.uk/ProductDetail/Molex/216990-0002?qs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
- C15: footprint SamacSys_Parts:CAPAE1030X1030N -> SamacSys_Parts:CAPC1005X55N
Connections:
- net +12V: now also J1.2
- net at PJ-057AH1.1: now also J1.1
Other:
- note removed: "PROBE OUTPUTS"
- moved on the sheet: PJ-057AH1
