File: HW/wled_V1/wled_V1.kicad_sch (KiCad schematic)
At the start: 29 parts, among them IC1 SN74AHCT125DR, J1 694106301002, K1 AHQSH112LM1F00G, Q1 MMBT3904-7-F

Commit message: route
Parts:
- added RN73H1JTTD1002F1: 10k, Resistor_SMD:R_0603_1608Metric_Pad0.98x0.95mm_HandSolder, symbol Device:R_Small
- added S1: TS14-1212-140-BK-160-SCR-D, SamacSys_Parts:TS0266160BK260LCRD, symbol SamacSys_Parts:TS14-1212-140-BK-160-SCR-D
- D1: footprint SOD3816X135N -> SamacSys_Parts:SOD3816X135N
- K1: footprint AHQSH112LM1F00G -> SamacSys_Parts:AHQSH112LM1F00G
- Q1: footprint SOT96P240X110-3N -> SamacSys_Parts:SOT96P240X110-3N
Connections:
- net +3.3V: now also RN73H1JTTD1002F1.2
- net GND: now also S1.3 (COM_1)
- net GPIO7: now reaches ESP32-S3-WROOM-1-N8.7 (GPIO7/TOUCH7/ADC1_CH6)
- net GPIO7: now also RN73H1JTTD1002F1.1, S1.1 (NO_1)
- no-connect marks 43 -> 44
Changed lines of the file:
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@@
   (junction (at 39.37 60.96) (diameter 0) (color 0 0 0 0)
   )
+  (junction (at 168.91 113.03) (diameter 0) (color 0 0 0 0)
+  )
   (junction (at 29.21 35.56) (diameter 0) (color 0 0 0 0)
   )
@@
   )
   (no_connect (at 267.97 64.77))
-  (no_connect (at 184.15 60.96))
   (no_connect (at 234.95 62.23))
   (no_connect (at 321.31 40.64))
@@
   (no_connect (at 87.63 93.98))
   (no_connect (at 179.07 99.06))
+  (no_connect (at 205.74 115.57))
   (no_connect (at 179.07 30.48))
   (no_connect (at 179.07 76.2))
@@
   (no_connect (at 179.07 27.94))
   (no_connect (at 87.63 99.06))
+  (no_connect (at 205.74 113.03))
   (no_connect (at 179.07 45.72))
   (no_connect (at 321.31 38.1))
@@
     (stroke (width 0) (type default))
   )
+  (wire (pts (xy 167.64 113.03) (xy 168.91 113.03))
+    (stroke (width 0) (type default))
+  )
   (wire (pts (xy 350.52 38.1) (xy 358.14 38.1))
+    (stroke (width 0) (type default))
+  )
+  (wire (pts (xy 168.91 113.03) (xy 175.26 113.03))
     (stroke (width 0) (type default))
   )
@@
   (text "POWER DISTRIBUTION\n" (at 14.605 17.145 0)
     (effects (font (size 2 2) (thickness 0.4) bold) (justify left bottom))
+  )
+  (global_label "GPIO7" (shape input) (at 184.15 60.96 0) (fields_autoplaced)
+    (effects (font (size 1.27 1.27)) (justify left))
+    (property "Intersheetrefs" "${INTERSHEET_REFS}" (at 192.7406 60.96 0)
+      (effects (font (size 1.27 1.27)) (justify left) hide)
+    )
   )
   (global_label "12v_commuted" (shape input) (at 344.17 75.565 0) (fields_autoplaced)
@@
     )
   )
+  (global_label "GPIO7" (shape input) (at 167.64 113.03 180) (fields_autoplaced)
+    (effects (font (size 1.27 1.27)) (justify right))
+    (property "Intersheetrefs" "${INTERSHEET_REFS}" (at 159.0494 113.03 0)
+      (effects (font (size 1.27 1.27)) (justify right) hide)
+    )
+  )
   (global_label "12v_commuted" (shape input) (at 349.885 45.72 180) (fields_autoplaced)
     (effects (font (size 1.27 1.27)) (justify right))
@@
         (path "/de2f0c7b-62aa-45a1-944c-ab4e5150c860"
           (reference "R2") (unit 1)
+        )
+      )
+    )
+  )
+  (symbol (lib_id "SamacSys_Parts:TS14-1212-140-BK-160-SCR-D") (at 175.26 113.03 0) (unit 1)
+    (in_bom yes) (on_board yes) (dnp no) (fields_autoplaced)
+    (property "Reference" "S1" (at 190.5 106.68 0)
+      (effects (font (size 1.27 1.27)))
+    )
+    (property "Value" "TS14-1212-140-BK-160-SCR-D" (at 190.5 109.22 0)
+      (effects (font (size 1.27 1.27)))
+    )
+    (property "Footprint" "SamacSys_Parts:TS0266160BK260LCRD" (at 201.93 207.95 0)
+      (effects (font (size 1.27 1.27)) (justify left top) hide)
+    )
+    (property "Datasheet" "https://www.cuidevices.com/product/resource/ts14.pdf" (at 201.93 307.95 0)
+      (effects (font (size 1.27 1.27)) (justify left top) hide)
+    )
+    (property "Height" "14.2" (at 201.93 507.95 0)
+      (effects (font (size 1.27 1.27)) (justify left top) hide)
+    )
+    (property "Mouser Part Number" "" (at 201.93 607.95 0)
+      (effects (font (size 1.27 1.27)) (justify left top) hide)
+    )
+    (property "Mouser Price/Stock" "" (at 201.93 707.95 0)
+      (effects (font (size 1.27 1.27)) (justify left top) hide)
+    )
+    (property "Manufacturer_Name" "CUI Devices" (at 201.93 807.95 0)
+      (effects (font (size 1.27 1.27)) (justify left top) hide)
+    )
+    (property "Manufacturer_Part_Number" "TS14-1212-140-BK-160-SCR-D" (at 201.93 907.95 0)
+      (effects (font (size 1.27 1.27)) (justify left top) hide)
+    )
+    (pin "1")
+    (pin "2")
+    (pin "3")
+    (pin "4")
+    (instances
+      (project "wled_V1"
+        (path "/de2f0c7b-62aa-45a1-944c-ab4e5150c860"
+          (reference "S1") (unit 1)
         )
       )
@@
     )
   )
+  (symbol (lib_id "power:GND") (at 175.26 115.57 270) (unit 1)
+    (in_bom yes) (on_board yes) (dnp no)
+    (property "Reference" "#PWR024" (at 168.91 115.57 0)
+      (effects (font (size 1.27 1.27)) hide)
+    )
+    (property "Value" "GND" (at 170.18 115.57 90)
+      (effects (font (size 1.27 1.27)))
+    )
+    (property "Footprint" "" (at 175.26 115.57 0)
+      (effects (font (size 1.27 1.27)) hide)
+    )
+    (property "Datasheet" "" (at 175.26 115.57 0)
+      (effects (font (size 1.27 1.27)) hide)
+    )
+    (pin "1")
+    (instances
+      (project "wled_V1"
+        (path "/de2f0c7b-62aa-45a1-944c-ab4e5150c860"
+          (reference "#PWR024") (unit 1)
+        )
+      )
+    )
+  )
   (symbol (lib_id "power:GND") (at 293.37 43.18 270) (unit 1)
     (in_bom yes) (on_board yes) (dnp no)
@@
         (path "/de2f0c7b-62aa-45a1-944c-ab4e5150c860"
           (reference "C13") (unit 1)
+        )
+      )
+    )
+  )
+  (symbol (lib_id "power:+3.3V") (at 168.91 107.95 0) (unit 1)
+    (in_bom yes) (on_board yes) (dnp no) (fields_autoplaced)
+    (property "Reference" "#PWR026" (at 168.91 111.76 0)
+      (effects (font (size 1.27 1.27)) hide)
+    )
+    (property "Value" "+3.3V" (at 168.91 104.14 0)
+      (effects (font (size 1.27 1.27)))
+    )
+    (property "Footprint" "" (at 168.91 107.95 0)
+      (effects (font (size 1.27 1.27)) hide)
+    )
+    (property "Datasheet" "" (at 168.91 107.95 0)
+      (effects (font (size 1.27 1.27)) hide)
+    )
+    (pin "1")
+    (instances
+      (project "wled_V1"
+        (path "/de2f0c7b-62aa-45a1-944c-ab4e5150c860"
+          (reference "#PWR026") (unit 1)
         )
       )
@@
     )
   )
+  (symbol (lib_id "Device:R_Small") (at 168.91 110.49 180) (unit 1)
+    (in_bom yes) (on_board yes) (dnp no)
+    (property "Reference" "RN73H1JTTD1002F1" (at 163.83 110.49 90)
+      (effects (font (size 1.27 1.27)) hide)
+    )
+    (property "Value" "10k" (at 170.18 110.49 0)
+      (effects (font (size 1.27 1.27)) (justify right))
+    )
+    (property "Footprint" "Resistor_SMD:R_0603_1608Metric_Pad0.98x0.95mm_HandSolder" (at 168.91 110.49 0)
+      (effects (font (size 1.27 1.27)) hide)
+    )
+    (property "Datasheet" "~" (at 168.91 110.49 0)
+      (effects (font (size 1.27 1.27)) hide)
+    )
+    (pin "1")
+    (pin "2")
+    (instances
+      (project "wled_V1"
+        (path "/de2f0c7b-62aa-45a1-944c-ab4e5150c860"
+          (reference "RN73H1JTTD1002F1") (unit 1)
+        )
+      )
+    )
+  )
   (symbol (lib_id "SamacSys_Parts:1N4148W_R1_00001") (at 302.26 67.945 270) (unit 1)
     (in_bom yes) (on_board yes) (dnp no)
@@
       (effects (font (size 1.27 1.27)) (justify left))
     )
-    (property "Footprint" "SOD3816X135N" (at 204.8 79.375 0)
+    (property "Footprint" "SamacSys_Parts:SOD3816X135N" (at 204.8 79.375 0)
       (effects (font (size 1.27 1.27)) (justify left top) hide)
     )
@@
       (effects (font (size 1.27 1.27)) (justify left))
     )
-    (property "Footprint" "SOT96P240X110-3N" (at 306.07 192.075 0)
+    (property "Footprint" "SamacSys_Parts:SOT96P240X110-3N" (at 306.07 192.075 0)
       (effects (font (size 1.27 1.27)) (justify left top) hide)
     )
@@
       (effects (font (size 1.27 1.27)))
     )
-    (property "Footprint" "AHQSH112LM1F00G" (at 340.36 167.945 0)
-      (effects (font (size 1.27 1.27)) (justify left top) hide)
-    )
+    (property "Footprint" "SamacSys_Parts:AHQSH112LM1F00G" (at 340.36 167.945 0)
+      (effects (font (size 1.27 1.27)) (justify left top) hide)
+    )
