File: HW/wled_V1/_autosave-wled_V1.kicad_sch (KiCad schematic)
At the start: 25 parts, among them J1 0031.8201, U3 TXS0102DCT

Commit message: Sourcing
Parts:
- AZ1117CR-3.3TRG1: footprint SamacSys_Parts:AZ1117CR33TRG1 -> Package_TO_SOT_SMD:TO-252-3_TabPin2
Changed lines of the file:
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@@
       (effects (font (size 1.27 1.27)))
     )
-    (property "Footprint" "SamacSys_Parts:AZ1117CR33TRG1" (at 39.37 27.94 0)
+    (property "Footprint" "Package_TO_SOT_SMD:TO-252-3_TabPin2" (at 39.37 27.94 0)
       (effects (font (size 1.27 1.27)) hide)
     )
@@
   (symbol (lib_id "SamacSys_Parts:216990-0002") (at 267.97 69.85 180) (unit 1)
     (in_bom yes) (on_board yes) (dnp no) (fields_autoplaced)
-    (property "Reference" "216990-0002" (at 251.46 40.64 0)
+    (property "Reference" "216990-0002" (at 251.46 39.37 0)
       (effects (font (size 1.27 1.27)))
     )
-    (property "Value" "USB_C_Receptacle" (at 251.46 43.18 0)
+    (property "Value" "USB_C_Receptacle" (at 251.46 41.91 0)
       (effects (font (size 1.27 1.27)))
     )
